Commit message: 1,add the read filepath automaticlly

File: Hector_ROS_Simulation/hector_description/urdf/hector_use_for_generate_jacobian.urdf (robot description, URDF)
Before this commit: robot hector_description, 30 links, 29 joints
Joints:
- joint L_foot_fixed_1: axis (none) -> 0 1 0; limit (none) -> lower=-1.4 upper=1.4 effort=33.5 velocity=21; type fixed -> revolute
- joint R_foot_fixed_1: axis (none) -> 0 1 0; limit (none) -> lower=-1.4 upper=1.4 effort=33.5 velocity=21; type fixed -> revolute
